File: IMU.kicad_sch (KiCad schematic)
At the start: 8 parts, among them U6 MPU-6050

Commit message: assigned footprints and checked the schematic
Parts:
- C16, C17, C18, C19: footprint (none) -> Capacitor_SMD:C_0402_1005Metric_Pad0.74x0.62mm_HandSolder
- JP1: footprint (none) -> Jumper:SolderJumper-2_P1.3mm_Open_RoundedPad1.0x1.5mm
- R11, R12: footprint (none) -> Resistor_SMD:R_0402_1005Metric_Pad0.72x0.64mm_HandSolder
Changed lines of the file:
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@@
       (effects (font (size 1.27 1.27)) (justify left))
     )
-    (property "Footprint" "" (at 150.8252 82.55 0)
+    (property "Footprint" "Capacitor_SMD:C_0402_1005Metric_Pad0.74x0.62mm_HandSolder" (at 150.8252 82.55 0)
       (effects (font (size 1.27 1.27)) hide)
     )
@@
       (effects (font (size 1.27 1.27)) (justify left))
     )
-    (property "Footprint" "" (at 182.5752 115.57 0)
+    (property "Footprint" "Capacitor_SMD:C_0402_1005Metric_Pad0.74x0.62mm_HandSolder" (at 182.5752 115.57 0)
       (effects (font (size 1.27 1.27)) hide)
     )
@@
       (effects (font (size 1.27 1.27)) (justify left))
     )
-    (property "Footprint" "" (at 97.028 87.63 90)
+    (property "Footprint" "Resistor_SMD:R_0402_1005Metric_Pad0.72x0.64mm_HandSolder" (at 97.028 87.63 90)
       (effects (font (size 1.27 1.27)) hide)
     )
@@
       (effects (font (size 1.27 1.27)) (justify left))
     )
-    (property "Footprint" "" (at 129.2352 82.55 0)
+    (property "Footprint" "Capacitor_SMD:C_0402_1005Metric_Pad0.74x0.62mm_HandSolder" (at 129.2352 82.55 0)
       (effects (font (size 1.27 1.27)) hide)
     )
@@
       (effects (font (size 1.27 1.27)) (justify left))
     )
-    (property "Footprint" "" (at 86.868 87.63 90)
+    (property "Footprint" "Resistor_SMD:R_0402_1005Metric_Pad0.72x0.64mm_HandSolder" (at 86.868 87.63 90)
       (effects (font (size 1.27 1.27)) hide)
     )
@@
       (effects (font (size 1.27 1.27)) (justify left))
     )
-    (property "Footprint" "" (at 166.0652 119.38 0)
+    (property "Footprint" "Capacitor_SMD:C_0402_1005Metric_Pad0.74x0.62mm_HandSolder" (at 166.0652 119.38 0)
       (effects (font (size 1.27 1.27)) hide)
     )
@@
       (effects (font (size 1 1)) (justify right))
     )
-    (property "Footprint" "" (at 114.3 106.68 0)
-      (effects (font (size 1.27 1.27)) hide)
-    )
+    (property "Footprint" "Jumper:SolderJumper-2_P1.3mm_Open_RoundedPad1.0x1.5mm" (at 114.3 106.68 0)
+      (effects (font (size 1.27 1.27)) hide)
+    )

Commit message: bottom board conn. done
Parts:
- removed R11, R12: 5.1k, Resistor_SMD:R_0402_1005Metric_Pad0.72x0.64mm_HandSolder, symbol Device:R
- JP1: footprint Jumper:SolderJumper-2_P1.3mm_Open_RoundedPad1.0x1.5mm -> Capacitor_SMD:C_0402_1005Metric
Changed lines of the file:
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@@
   (junction (at 143.51 73.66) (diameter 0) (color 0 0 0 0)
   )
-  (junction (at 109.22 93.98) (diameter 0) (color 0 0 0 0)
-  )
   (junction (at 121.92 109.22) (diameter 0) (color 0 0 0 0)
-  )
-  (junction (at 104.14 96.52) (diameter 0) (color 0 0 0 0)
   )
   (junction (at 140.97 73.66) (diameter 0) (color 0 0 0 0)
@@
     (stroke (width 0) (type default))
   )
-  (wire (pts (xy 85.09 93.98) (xy 109.22 93.98))
-    (stroke (width 0) (type default))
-  )
   (wire (pts (xy 165.1 109.22) (xy 165.1 111.76))
     (stroke (width 0) (type default))
@@
     (stroke (width 0) (type default))
   )
-  (wire (pts (xy 85.09 82.55) (xy 85.09 83.82))
-    (stroke (width 0) (type default))
-  )
   (wire (pts (xy 140.97 69.85) (xy 140.97 73.66))
     (stroke (width 0) (type default))
@@
     (stroke (width 0) (type default))
   )
-  (wire (pts (xy 85.09 91.44) (xy 85.09 93.98))
-    (stroke (width 0) (type default))
-  )
-  (wire (pts (xy 95.25 82.55) (xy 95.25 83.82))
-    (stroke (width 0) (type default))
-  )
   (wire (pts (xy 172.72 93.98) (xy 158.75 93.98))
     (stroke (width 0) (type default))
   )
-  (wire (pts (xy 95.25 96.52) (xy 104.14 96.52))
-    (stroke (width 0) (type default))
-  )
   (wire (pts (xy 104.14 96.52) (xy 123.19 96.52))
-    (stroke (width 0) (type default))
-  )
-  (wire (pts (xy 95.25 91.44) (xy 95.25 96.52))
     (stroke (width 0) (type default))
   )
@@
     )
   )
-  (symbol (lib_id "power:+3V3") (at 95.25 82.55 0) (unit 1)
-    (in_bom yes) (on_board yes) (dnp no) (fields_autoplaced)
-    (property "Reference" "#PWR08" (at 95.25 86.36 0)
-      (effects (font (size 1.27 1.27)) hide)
-    )
-    (property "Value" "+3V3" (at 95.25 77.47 0)
-      (effects (font (size 1.27 1.27)))
-    )
-    (property "Footprint" "" (at 95.25 82.55 0)
-      (effects (font (size 1.27 1.27)) hide)
-    )
-    (property "Datasheet" "" (at 95.25 82.55 0)
-      (effects (font (size 1.27 1.27)) hide)
-    )
-    (pin "1")
-    (instances
-      (project "RP2040_SOS_band"
-        (path "/1d911b84-17e1-4d47-ac8f-a730104b53ed"
-          (reference "#PWR08") (unit 1)
-        )
-        (path "/1d911b84-17e1-4d47-ac8f-a730104b53ed/892de33d-264e-4bda-a61c-c8174f81e463"
-          (reference "#PWR06") (unit 1)
-        )
-        (path "/1d911b84-17e1-4d47-ac8f-a730104b53ed/afb52c89-42a1-49e5-9806-4765b2ea4612"
-          (reference "#PWR033") (unit 1)
-        )
-      )
-    )
-  )
   (symbol (lib_id "power:GND") (at 128.27 83.82 0) (unit 1)
     (in_bom yes) (on_board yes) (dnp no) (fields_autoplaced)
@@
     )
   )
-  (symbol (lib_id "Device:R") (at 95.25 87.63 180) (unit 1)
-    (in_bom yes) (on_board yes) (dnp no) (fields_autoplaced)
-    (property "Reference" "R12" (at 92.71 88.265 0)
-      (effects (font (size 1.27 1.27)) (justify left))
-    )
-    (property "Value" "5.1k" (at 92.71 85.725 0)
-      (effects (font (size 1.27 1.27)) (justify left))
-    )
-    (property "Footprint" "Resistor_SMD:R_0402_1005Metric_Pad0.72x0.64mm_HandSolder" (at 97.028 87.63 90)
-      (effects (font (size 1.27 1.27)) hide)
-    )
-    (property "Datasheet" "~" (at 95.25 87.63 0)
+  (symbol (lib_id "Device:C") (at 128.27 78.74 0) (unit 1)
+    (in_bom yes) (on_board yes) (dnp no) (fields_autoplaced)
+    (property "Reference" "C18" (at 132.08 78.105 0)
+      (effects (font (size 1.27 1.27)) (justify left))
+    )
+    (property "Value" "0.1uF" (at 132.08 80.645 0)
+      (effects (font (size 1.27 1.27)) (justify left))
+    )
+    (property "Footprint" "Capacitor_SMD:C_0402_1005Metric_Pad0.74x0.62mm_HandSolder" (at 129.2352 82.55 0)
+      (effects (font (size 1.27 1.27)) hide)
+    )
+    (property "Datasheet" "~" (at 128.27 78.74 0)
       (effects (font (size 1.27 1.27)) hide)
     )
@@
       (project "RP2040_SOS_band"
         (path "/1d911b84-17e1-4d47-ac8f-a730104b53ed/afb52c89-42a1-49e5-9806-4765b2ea4612"
-          (reference "R12") (unit 1)
-        )
-      )
-    )
-  )
-  (symbol (lib_id "Device:C") (at 128.27 78.74 0) (unit 1)
-    (in_bom yes) (on_board yes) (dnp no) (fields_autoplaced)
-    (property "Reference" "C18" (at 132.08 78.105 0)
-      (effects (font (size 1.27 1.27)) (justify left))
-    )
-    (property "Value" "0.1uF" (at 132.08 80.645 0)
-      (effects (font (size 1.27 1.27)) (justify left))
-    )
-    (property "Footprint" "Capacitor_SMD:C_0402_1005Metric_Pad0.74x0.62mm_HandSolder" (at 129.2352 82.55 0)
-      (effects (font (size 1.27 1.27)) hide)
-    )
-    (property "Datasheet" "~" (at 128.27 78.74 0)
-      (effects (font (size 1.27 1.27)) hide)
-    )
-    (pin "1")
-    (pin "2")
-    (instances
-      (project "RP2040_SOS_band"
-        (path "/1d911b84-17e1-4d47-ac8f-a730104b53ed/afb52c89-42a1-49e5-9806-4765b2ea4612"
           (reference "C18") (unit 1)
         )
@@
     )
   )
-  (symbol (lib_id "Device:R") (at 85.09 87.63 180) (unit 1)
-    (in_bom yes) (on_board yes) (dnp no) (fields_autoplaced)
-    (property "Reference" "R11" (at 82.55 88.265 0)
-      (effects (font (size 1.27 1.27)) (justify left))
-    )
-    (property "Value" "5.1k" (at 82.55 85.725 0)
-      (effects (font (size 1.27 1.27)) (justify left))
-    )
-    (property "Footprint" "Resistor_SMD:R_0402_1005Metric_Pad0.72x0.64mm_HandSolder" (at 86.868 87.63 90)
-      (effects (font (size 1.27 1.27)) hide)
-    )
-    (property "Datasheet" "~" (at 85.09 87.63 0)
-      (effects (font (size 1.27 1.27)) hide)
-    )
-    (pin "1")
-    (pin "2")
-    (instances
-      (project "RP2040_SOS_band"
-        (path "/1d911b84-17e1-4d47-ac8f-a730104b53ed/afb52c89-42a1-49e5-9806-4765b2ea4612"
-          (reference "R11") (unit 1)
-        )
-      )
-    )
-  )
   (symbol (lib_id "power:GND") (at 140.97 120.65 0) (unit 1)
     (in_bom yes) (on_board yes) (dnp no) (fields_autoplaced)
@@
         (path "/1d911b84-17e1-4d47-ac8f-a730104b53ed/afb52c89-42a1-49e5-9806-4765b2ea4612"
           (reference "#PWR031") (unit 1)
-        )
-      )
-    )
-  )
-  (symbol (lib_id "power:+3V3") (at 85.09 82.55 0) (unit 1)
-    (in_bom yes) (on_board yes) (dnp no) (fields_autoplaced)
-    (property "Reference" "#PWR08" (at 85.09 86.36 0)
-      (effects (font (size 1.27 1.27)) hide)
-    )
-    (property "Value" "+3V3" (at 85.09 77.47 0)
-      (effects (font (size 1.27 1.27)))
-    )
-    (property "Footprint" "" (at 85.09 82.55 0)
-      (effects (font (size 1.27 1.27)) hide)
-    )
-    (property "Datasheet" "" (at 85.09 82.55 0)
-      (effects (font (size 1.27 1.27)) hide)
-    )
-    (pin "1")
-    (instances
-      (project "RP2040_SOS_band"
-        (path "/1d911b84-17e1-4d47-ac8f-a730104b53ed"
-          (reference "#PWR08") (unit 1)
-        )
-        (path "/1d911b84-17e1-4d47-ac8f-a730104b53ed/892de33d-264e-4bda-a61c-c8174f81e463"
-          (reference "#PWR06") (unit 1)
-        )
-        (path "/1d911b84-17e1-4d47-ac8f-a730104b53ed/afb52c89-42a1-49e5-9806-4765b2ea4612"
-          (reference "#PWR028") (unit 1)
         )
       )
@@
       (effects (font (size 1 1)) (justify right))
     )
-    (property "Footprint" "Jumper:SolderJumper-2_P1.3mm_Open_RoundedPad1.0x1.5mm" (at 114.3 106.68 0)
-      (effects (font (size 1.27 1.27)) hide)
-    )
+    (property "Footprint" "Capacitor_SMD:C_0402_1005Metric" (at 114.3 106.68 0)
+      (effects (font (size 1.27 1.27)) hide)
+    )
