File: RP2040_SOS_band.kicad_sch (KiCad schematic)
At the start: 0 parts

Commit message: bottom board conn. done
Other:
- sheet ATGM336H renamed Quectel L96
Changed lines of the file:
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@@
     (stroke (width 0.1524) (type solid))
     (fill (color 0 0 0 0.0000))
-    (property "Sheetname" "ATGM336H" (at 118.11 64.0584 0)
+    (property "Sheetname" "Quectel L96" (at 118.11 64.0584 0)
       (effects (font (size 1.27 1.27)) (justify left bottom))
     )
