File: connectors.kicad_sch (KiCad schematic)
At the start: 2 parts, among them J4 10Pin FPC Bottom board, J4 10Pin FPC TOP Board

Commit message: assigned footprints and checked the schematic
Parts:
- J4: footprint (none) -> 10 Pin FPC:686110183522
Changed lines of the file:
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@@
       (effects (font (size 1.27 1.27)) (justify left))
     )
-    (property "Footprint" "" (at 118.11 113.03 0)
+    (property "Footprint" "10 Pin FPC:686110183522" (at 118.11 113.03 0)
       (effects (font (size 1.27 1.27)) hide)
     )
@@
       (effects (font (size 1.27 1.27)) (justify left))
     )
-    (property "Footprint" "" (at 162.56 113.03 0)
+    (property "Footprint" "10 Pin FPC:686110183522" (at 162.56 113.03 0)
       (effects (font (size 1.27 1.27)) hide)
     )

Commit message: bottom board conn. done
Connections:
- net GPS_RXD: no longer J4.5 (Pin_5)
- net GPS_TXD: now also J4.6 (Pin_6); no longer J4.4 (Pin_4), J4.4 (Pin_4)
- net GSM_RX: now also J4.1 (Pin_1); no longer J4.8 (Pin_8), J4.8 (Pin_8)
- net GSM_TX: now also J4.2 (Pin_2); no longer J4.7 (Pin_7), J4.7 (Pin_7)
- net PWR_KEY_GSM: now also J4.4 (Pin_4); no longer J4.2 (Pin_2), J4.2 (Pin_2)
- net VDD_3.3: no longer J4.9 (Pin_9)
- net +3V3 renamed GSM_RX_t
- net GSM_RX_t: no longer J4.1 (Pin_1)
- net GPS_PPS renamed GPS_TXD_t
- net GPS_TXD_t: no longer J4.6 (Pin_6)
- net GPS_RST renamed Force_ON
- net Force_ON: no longer J4.3 (Pin_3)
- new net Force_ON_t: J4.3 (Pin_3)
- new net GPS_RXD_t: J4.5 (Pin_5)
- new net GSM_TX_t: J4.2 (Pin_2)
- new net PWR_KEY_GSM_t: J4.4 (Pin_4)
- new net VDD_3.3_t: J4.9 (Pin_9)
- no-connect marks 0 -> 4
