File: RP2040.kicad_sch (KiCad schematic)
At the start: 31 parts, among them J1 TYPE_C-31M12, SW1 Boot, U1 RP2040, U2 W25Q32JVSS, Y1 Crystal_GND24

Commit message: assigned footprints and checked the schematic
Parts:
- added SW1: PWR, TS24CA Tactile switch:TS24CA, symbol Switch:SW_Push
- added SW1: UP, TS24CA Tactile switch:TS24CA, symbol Switch:SW_Push
- added SW1: NAV, TS24CA Tactile switch:TS24CA, symbol Switch:SW_Push
- SW1: footprint (none) -> TS24CA Tactile switch:TS24CA
- TP3, TP4, TP5, TP6: footprint (none) -> TestPoint:TestPoint_Pad_D2.0mm
Connections:
- net GND: now also SW1.1, SW1.1, SW1.1
- net NAV_BUTTON: now also SW1.2
- net PWR_BUTTON: now also SW1.2
- net UP_BUTTON: now also SW1.2
Changed lines of the file:
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@@
+    (stroke (width 0) (type default))
+  )
+  (wire (pts (xy 143.51 34.29) (xy 147.32 34.29))
     (stroke (width 0) (type default))
   )
@@
     (stroke (width 0) (type default))
   )
+  (wire (pts (xy 143.51 35.56) (xy 143.51 34.29))
+    (stroke (width 0) (type default))
+  )
   (wire (pts (xy 102.87 167.64) (xy 114.3 167.64))
     (stroke (width 0) (type default))
@@
     (stroke (width 0) (type default))
   )
+  (wire (pts (xy 143.51 52.07) (xy 147.32 52.07))
+    (stroke (width 0) (type default))
+  )
   (wire (pts (xy 29.21 177.8) (xy 29.21 181.61))
     (stroke (width 0) (type default))
@@
     (stroke (width 0) (type default))
   )
+  (wire (pts (xy 143.51 67.31) (xy 143.51 66.04))
+    (stroke (width 0) (type default))
+  )
   (wire (pts (xy 73.66 35.56) (xy 73.66 36.83))
     (stroke (width 0) (type default))
@@
     (stroke (width 0) (type default))
   )
+  (wire (pts (xy 143.51 53.34) (xy 143.51 52.07))
+    (stroke (width 0) (type default))
+  )
   (wire (pts (xy 158.75 153.67) (xy 158.75 152.4))
     (stroke (width 0) (type default))
@@
   )
   (wire (pts (xy 43.18 55.88) (xy 43.18 54.61))
+    (stroke (width 0) (type default))
+  )
+  (wire (pts (xy 143.51 66.04) (xy 147.32 66.04))
     (stroke (width 0) (type default))
   )
@@
     )
   )
+  (global_label "UP_BUTTON" (shape output) (at 157.48 66.04 0) (fields_autoplaced)
+    (effects (font (size 1 1) (color 0 132 0 1)) (justify left))
+    (property "Intersheetrefs" "${INTERSHEET_REFS}" (at 168.244 66.04 0)
+      (effects (font (size 1.27 1.27)) (justify left) hide)
+    )
+  )
   (global_label "D-" (shape input) (at 236.22 40.64 0) (fields_autoplaced)
     (effects (font (face "Century Gothic") (size 1 1)) (justify left))
@@
     )
   )
+  (global_label "NAV_BUTTON" (shape output) (at 157.48 52.07 0) (fields_autoplaced)
+    (effects (font (size 1 1) (color 0 132 0 1)) (justify left))
+    (property "Intersheetrefs" "${INTERSHEET_REFS}" (at 168.9582 52.07 0)
+      (effects (font (size 1.27 1.27)) (justify left) hide)
+    )
+  )
+  (global_label "PWR_BUTTON" (shape output) (at 157.48 34.29 0) (fields_autoplaced)
+    (effects (font (size 1 1) (color 0 132 0 1)) (justify left))
+    (property "Intersheetrefs" "${INTERSHEET_REFS}" (at 169.3393 34.29 0)
+      (effects (font (size 1.27 1.27)) (justify left) hide)
+    )
+  )
   (global_label "SDA_OLED" (shape output) (at 97.79 49.53 0) (fields_autoplaced)
     (effects (font (size 1 1) (color 0 132 0 1)) (justify left))
@@
       (effects (font (size 1.27 1.27)) (justify left))
     )
-    (property "Footprint" "" (at 163.83 152.4 0)
+    (property "Footprint" "TestPoint:TestPoint_Pad_D2.0mm" (at 163.83 152.4 0)
       (effects (font (size 1.27 1.27)) hide)
     )
@@
     )
   )
+  (symbol (lib_id "power:GND") (at 143.51 67.31 0) (unit 1)
+    (in_bom yes) (on_board yes) (dnp no)
+    (property "Reference" "#PWR016" (at 143.51 73.66 0)
+      (effects (font (size 1.27 1.27)) hide)
+    )
+    (property "Value" "GND" (at 147.32 69.85 0)
+      (effects (font (size 1.27 1.27)) hide)
+    )
+    (property "Footprint" "" (at 143.51 67.31 0)
+      (effects (font (size 1.27 1.27)) hide)
+    )
+    (property "Datasheet" "" (at 143.51 67.31 0)
+      (effects (font (size 1.27 1.27)) hide)
+    )
+    (pin "1")
+    (instances
+      (project "RP2040_SOS_band"
+        (path "/1d911b84-17e1-4d47-ac8f-a730104b53ed"
+          (reference "#PWR016") (unit 1)
+        )
+        (path "/1d911b84-17e1-4d47-ac8f-a730104b53ed/892de33d-264e-4bda-a61c-c8174f81e463"
+          (reference "#PWR080") (unit 1)
+        )
+      )
+    )
+  )
   (symbol (lib_id "Device:C") (at 102.87 175.26 0) (unit 1)
     (in_bom yes) (on_board yes) (dnp no) (fields_autoplaced)
@@
       (effects (font (size 1.27 1.27)) (justify left))
     )
-    (property "Footprint" "" (at 176.53 152.4 0)
+    (property "Footprint" "TestPoint:TestPoint_Pad_D2.0mm" (at 176.53 152.4 0)
       (effects (font (size 1.27 1.27)) hide)
     )
@@
     )
   )
+  (symbol (lib_id "Switch:SW_Push") (at 152.4 34.29 0) (unit 1)
+    (in_bom yes) (on_board yes) (dnp no) (fields_autoplaced)
+    (property "Reference" "SW1" (at 152.4 27.94 0)
+      (effects (font (size 1.27 1.27)))
+    )
+    (property "Value" "PWR" (at 152.4 30.48 0)
+      (effects (font (size 1.27 1.27)))
+    )
+    (property "Footprint" "TS24CA Tactile switch:TS24CA" (at 152.4 29.21 0)
+      (effects (font (size 1.27 1.27)) hide)
+    )
+    (property "Datasheet" "~" (at 152.4 29.21 0)
+      (effects (font (size 1.27 1.27)) hide)
+    )
+    (pin "1")
+    (pin "2")
+    (instances
+      (project "RP2040_SOS_band"
+        (path "/1d911b84-17e1-4d47-ac8f-a730104b53ed"
+          (reference "SW1") (unit 1)
+        )
+        (path "/1d911b84-17e1-4d47-ac8f-a730104b53ed/892de33d-264e-4bda-a61c-c8174f81e463"
+          (reference "SW2") (unit 1)
+        )
+      )
+    )
+  )
   (symbol (lib_id "Device:Crystal_GND24") (at 232.41 101.6 0) (unit 1)
     (in_bom yes) (on_board yes) (dnp no)
@@
     )
   )
+  (symbol (lib_id "Switch:SW_Push") (at 152.4 66.04 0) (unit 1)
+    (in_bom yes) (on_board yes) (dnp no) (fields_autoplaced)
+    (property "Reference" "SW1" (at 152.4 59.69 0)
+      (effects (font (size 1.27 1.27)))
+    )
+    (property "Value" "UP" (at 152.4 62.23 0)
+      (effects (font (size 1.27 1.27)))
+    )
+    (property "Footprint" "TS24CA Tactile switch:TS24CA" (at 152.4 60.96 0)
+      (effects (font (size 1.27 1.27)) hide)
+    )
+    (property "Datasheet" "~" (at 152.4 60.96 0)
+      (effects (font (size 1.27 1.27)) hide)
+    )
+    (pin "1")
+    (pin "2")
+    (instances
+      (project "RP2040_SOS_band"
+        (path "/1d911b84-17e1-4d47-ac8f-a730104b53ed"
+          (reference "SW1") (unit 1)
+        )
+        (path "/1d911b84-17e1-4d47-ac8f-a730104b53ed/892de33d-264e-4bda-a61c-c8174f81e463"
+          (reference "SW4") (unit 1)
+        )
+      )
+    )
+  )
   (symbol (lib_id "Device:R") (at 254 41.91 0) (unit 1)
     (in_bom yes) (on_board yes) (dnp no)
@@
       (effects (font (size 1.27 1.27)))
     )
-    (property "Footprint" "" (at 144.78 86.36 0)
+    (property "Footprint" "TS24CA Tactile switch:TS24CA" (at 144.78 86.36 0)
       (effects (font (size 1.27 1.27)) hide)
     )
@@
     )
   )
+  (symbol (lib_id "power:GND") (at 143.51 35.56 0) (unit 1)
+    (in_bom yes) (on_board yes) (dnp no)
+    (property "Reference" "#PWR016" (at 143.51 41.91 0)
+      (effects (font (size 1.27 1.27)) hide)
+    )
+    (property "Value" "GND" (at 147.32 38.1 0)
+      (effects (font (size 1.27 1.27)) hide)
+    )
+    (property "Footprint" "" (at 143.51 35.56 0)
+      (effects (font (size 1.27 1.27)) hide)
+    )
+    (property "Datasheet" "" (at 143.51 35.56 0)
+      (effects (font (size 1.27 1.27)) hide)
+    )
+    (pin "1")
+    (instances
+      (project "RP2040_SOS_band"
+        (path "/1d911b84-17e1-4d47-ac8f-a730104b53ed"
+          (reference "#PWR016") (unit 1)
+        )
+        (path "/1d911b84-17e1-4d47-ac8f-a730104b53ed/892de33d-264e-4bda-a61c-c8174f81e463"
+          (reference "#PWR051") (unit 1)
+        )
+      )
+    )
+  )
+  (symbol (lib_id "Switch:SW_Push") (at 152.4 52.07 0) (unit 1)
+    (in_bom yes) (on_board yes) (dnp no) (fields_autoplaced)
+    (property "Reference" "SW1" (at 152.4 45.72 0)
+      (effects (font (size 1.27 1.27)))
+    )
+    (property "Value" "NAV" (at 152.4 48.26 0)
+      (effects (font (size 1.27 1.27)))
+    )
+    (property "Footprint" "TS24CA Tactile switch:TS24CA" (at 152.4 46.99 0)
+      (effects (font (size 1.27 1.27)) hide)
+    )
+    (property "Datasheet" "~" (at 152.4 46.99 0)
+      (effects (font (size 1.27 1.27)) hide)
+    )
+    (pin "1")
+    (pin "2")
+    (instances
+      (project "RP2040_SOS_band"
+        (path "/1d911b84-17e1-4d47-ac8f-a730104b53ed"
+          (reference "SW1") (unit 1)
+        )
+        (path "/1d911b84-17e1-4d47-ac8f-a730104b53ed/892de33d-264e-4bda-a61c-c8174f81e463"
+          (reference "SW3") (unit 1)
+        )
+      )
+    )
+  )
   (symbol (lib_id "Device:R") (at 247.65 45.72 180) (unit 1)
     (in_bom yes) (on_board yes) (dnp no)
@@
       (effects (font (size 1.27 1.27)) (justify left))
     )
-    (property "Footprint" "" (at 172.72 152.4 0)
+    (property "Footprint" "TestPoint:TestPoint_Pad_D2.0mm" (at 172.72 152.4 0)
       (effects (font (size 1.27 1.27)) hide)
     )
@@
       (effects (font (size 1.27 1.27)) (justify left))
     )
-    (property "Footprint" "" (at 167.64 152.4 0)
+    (property "Footprint" "TestPoint:TestPoint_Pad_D2.0mm" (at 167.64 152.4 0)
       (effects (font (size 1.27 1.27)) hide)
     )
@@
         )
       )
+    )
+  )
+  (symbol (lib_id "power:GND") (at 143.51 53.34 0) (unit 1)
+    (in_bom yes) (on_board yes) (dnp no)
+    (property "Reference" "#PWR016" (at 143.51 59.69 0)
+      (effects (font (size 1.27 1.27)) hide)
+    )
+    (property "Value" "GND" (at 147.32 55.88 0)
+      (effects (font (size 1.27 1.27)) hide)
+    )
+    (property "Footprint" "" (at 143.51 53.34 0)
+      (effects (font (size 1.27 1.27)) hide)
+    )
+    (property "Datasheet" "" (at 143.51 53.34 0)
+      (effects (font (size 1.27 1.27)) hide)
+    )
+    (pin "1")
+    (instances
+      (project "RP2040_SOS_band"
+        (path "/1d911b84-17e1-4d47-ac8f-a730104b53ed"
+          (reference "#PWR016") (unit 1)
+        )
+        (path "/1d911b84-17e1-4d47-ac8f-a730104b53ed/892de33d-264e-4bda-a61c-c8174f81e463"
+          (reference "#PWR079") (unit 1)
+        )
+      )

Commit message: bottom board conn. done
Parts:
- removed SW1: UP, TS24CA Tactile switch:TS24CA, symbol Switch:SW_Push
- added R11: DNP/TP, Resistor_SMD:R_0402_1005Metric_Pad0.72x0.64mm_HandSolder, symbol Device:R
- D2: footprint LED_SMD:LED_0805_2012Metric_Pad1.15x1.40mm_HandSolder -> LED_SMD:LED_0402_1005Metric_Pad0.77x0.64mm_HandSolder
- TP3, TP4, TP5, TP6: footprint TestPoint:TestPoint_Pad_D2.0mm -> TestPoint:TestPoint_Pad_D1.0mm
- U2: footprint Package_SO:SOIC-8_5.23x5.23mm_P1.27mm -> Package_SON:WSON-8-1EP_6x5mm_P1.27mm_EP3.4x4.3mm
Connections:
- net GPS_PPS is gone; now on net MPU_INT: U1.35 (GPIO23)
- net CHARGER_EN: now also U1.38 (GPIO26_ADC0); no longer U1.40 (GPIO28_ADC2)
- net GND: now also R11.1
- net GPS_RXD: now also U1.31 (GPIO20); no longer U1.36 (GPIO24)
- net GPS_TXD: now also U1.32 (GPIO21); no longer U1.37 (GPIO25)
- net Heart_rate_INT: now also U1.13 (GPIO10); no longer U1.14 (GPIO11)
- net MAX30102_SCL: now also U1.37 (GPIO25); no longer U1.12 (GPIO9)
- net MAX30102_SDA: now also U1.36 (GPIO24); no longer U1.11 (GPIO8)
- net MPU_INT: no longer U1.16 (GPIO13)
- net NAV_BUTTON: now also U1.17 (GPIO14); no longer U1.31 (GPIO20)
- net PWR_BUTTON: now also U1.3 (GPIO1); no longer U1.29 (GPIO18)
- net VBUS: no longer R8.2
- net V_SENSE: now also U1.41 (GPIO29_ADC3); no longer U1.38 (GPIO26_ADC0)
- net at R1.1: now also R11.2; no longer SW1.2
- net NAV_BUTTON_2: now reaches U1.2 (GPIO0)
- net NAV_BUTTON_2: now also SW1.2
- net PWR_KEY_GSM: now reaches U1.30 (GPIO19)
- net GPS_RST: no longer names the net of U1.9 (GPIO7)
- net LDO_EN: no longer names the net of U1.8 (GPIO6)
- net UP_BUTTON: no longer names the net of U1.34 (GPIO22)
- new net Force_ON: U1.29 (GPIO18)
- new net Onboard_LED: R8.2, U1.14 (GPIO11)
Other:
- moved on the sheet: SW1, TP3, U2

Commit message: Final Design
Parts:
- SW1: footprint TS24CA Tactile switch:TS24CA -> TL3330AF260QG:SW_TL3330AF260QG
- SW1: value Boot -> NAV2; footprint TS24CA Tactile switch:TS24CA -> TL3330AF260QG:SW_TL3330AF260QG
Changed lines of the file:
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@@
       (effects (font (size 1.27 1.27)))
     )
-    (property "Footprint" "TS24CA Tactile switch:TS24CA" (at 152.4 29.21 0)
+    (property "Footprint" "TL3330AF260QG:SW_TL3330AF260QG" (at 152.4 29.21 0)
       (effects (font (size 1.27 1.27)) hide)
     )
@@
       (effects (font (size 1.27 1.27)))
     )
-    (property "Value" "Boot" (at 151.13 60.96 0)
-      (effects (font (size 1.27 1.27)))
-    )
-    (property "Footprint" "TS24CA Tactile switch:TS24CA" (at 151.13 59.69 0)
+    (property "Value" "NAV2" (at 151.13 60.96 0)
+      (effects (font (size 1.27 1.27)))
+    )
+    (property "Footprint" "TL3330AF260QG:SW_TL3330AF260QG" (at 151.13 59.69 0)
       (effects (font (size 1.27 1.27)) hide)
     )
@@
       (effects (font (size 1.27 1.27)))
     )
-    (property "Footprint" "TS24CA Tactile switch:TS24CA" (at 152.4 46.99 0)
-      (effects (font (size 1.27 1.27)) hide)
-    )
+    (property "Footprint" "TL3330AF260QG:SW_TL3330AF260QG" (at 152.4 46.99 0)
+      (effects (font (size 1.27 1.27)) hide)
+    )
