File: RP2040_SOS_band.kicad_pcb (KiCad board)
At the start: 2 copper layers, 39 parts, among them IC1 ATGM336H-5N31, J1 TYPE_C-31M12, J2 SIM8060-6-0-14-00-A, U1 RP2040, U10 M66, U2 AP1117-33, U3 W25Q32JVSS, U4 MAX30102, U5 MCP73831-2-OT, U6 MPU-6050, U8 3.3V EN_LDO, U9 M24C32, Y1 Crystal_GND24

Commit message: assigned footprints and checked the schematic
Parts:
- removed BT1: 1220, CR1220 Cell:CH291-1220LF
- added ANT1: 1462350001, Molex GPS antenna:ANT_1462350001, F.Cu at (234.6, 91.7)
- added C15: 10uF, Capacitor_SMD:C_0402_1005Metric_Pad0.74x0.62mm_HandSolder, F.Cu at (239.7, 90.1)
- added C16: 0.1uF, Capacitor_SMD:C_0402_1005Metric_Pad0.74x0.62mm_HandSolder, F.Cu at (232.7, 100.0)
- added C17: 2.2nF, Capacitor_SMD:C_0402_1005Metric_Pad0.74x0.62mm_HandSolder, F.Cu at (232.7, 102.0)
- added C18: 0.1uF, Capacitor_SMD:C_0402_1005Metric_Pad0.74x0.62mm_HandSolder, F.Cu at (232.7, 104.0)
- added C19: 0.1uF, Capacitor_SMD:C_0402_1005Metric_Pad0.74x0.62mm_HandSolder, F.Cu at (232.7, 105.9)
- added C20: 0.1uF, Capacitor_SMD:C_0402_1005Metric_Pad0.74x0.62mm_HandSolder, F.Cu at (244.4, 100.0)
- added C21: 10uF, Capacitor_SMD:C_0402_1005Metric_Pad0.74x0.62mm_HandSolder, F.Cu at (221.8, 126.1)
- added C22: 10uF, Capacitor_SMD:C_0402_1005Metric_Pad0.74x0.62mm_HandSolder, F.Cu at (241.4, 79.7)
- added C24: 30pF, Capacitor_SMD:C_0402_1005Metric_Pad0.74x0.62mm_HandSolder, F.Cu at (218.5, 90.1)
- added C25: 30pF, Capacitor_SMD:C_0402_1005Metric_Pad0.74x0.62mm_HandSolder, F.Cu at (218.5, 92.1)
- added C26: 30pF, Capacitor_SMD:C_0402_1005Metric_Pad0.74x0.62mm_HandSolder, F.Cu at (218.5, 94.1)
- added C27: 30pF, Capacitor_SMD:C_0402_1005Metric_Pad0.74x0.62mm_HandSolder, F.Cu at (218.5, 96.0)
- added C28: 100nF, Capacitor_SMD:C_0402_1005Metric_Pad0.74x0.62mm_HandSolder, F.Cu at (218.5, 98.0)
- added C29: 470uF, Capacitor_Tantalum_SMD:CP_EIA-7343-30_AVX-N, F.Cu at (218.5, 100.0)
- added C30: 100nF, Capacitor_SMD:C_0402_1005Metric_Pad0.74x0.62mm_HandSolder, F.Cu at (221.7, 90.1)
- added C31: 30pF, Capacitor_SMD:C_0402_1005Metric_Pad0.74x0.62mm_HandSolder, F.Cu at (221.7, 92.1)
- added C32: NC, Capacitor_SMD:C_0402_1005Metric_Pad0.74x0.62mm_HandSolder, F.Cu at (221.7, 94.1)
- added C33: NC, Capacitor_SMD:C_0402_1005Metric_Pad0.74x0.62mm_HandSolder, F.Cu at (221.7, 96.0)
- added C34: NC, Capacitor_SMD:C_0402_1005Metric_Pad0.74x0.62mm_HandSolder, F.Cu at (239.7, 92.1)
- added C35: NC, Capacitor_SMD:C_0402_1005Metric_Pad0.74x0.62mm_HandSolder, F.Cu at (239.7, 94.1)
- added J3: 10Pin FPC TOP Board, 10 Pin FPC:686110183522, F.Cu at (225.7, 78.2)
- added J4: 10Pin FPC Bottom board, 10 Pin FPC:686110183522, F.Cu at (225.7, 84.2)
- added J5: U.FL-R-SMT-1(10), U.FL-R-SMT-1_10_:HRS_U.FL-R-SMT-1(10), F.Cu at (226.2, 99.2)
- added JP1: I2C address change, Jumper:SolderJumper-2_P1.3mm_Open_RoundedPad1.0x1.5mm, F.Cu at (222.3, 139.0)
- added L1: 47nH, Inductor_SMD:L_0402_1005Metric, F.Cu at (235.8, 96.0)
- added Q1: HSSN3134, Package_TO_SOT_SMD:SOT-323_SC-70, F.Cu at (242.0, 76.9)
- added R10: 2.2k, Resistor_SMD:R_0402_1005Metric_Pad0.72x0.64mm_HandSolder, F.Cu at (238.2, 76.1)
- added R11: 5.1k, Resistor_SMD:R_0402_1005Metric_Pad0.72x0.64mm_HandSolder, F.Cu at (236.0, 100.0)
- added R12: 5.1k, Resistor_SMD:R_0402_1005Metric_Pad0.72x0.64mm_HandSolder, F.Cu at (236.0, 102.0)
- added R13: 10k, Resistor_SMD:R_0402_1005Metric_Pad0.72x0.64mm_HandSolder, F.Cu at (238.2, 78.1)
- added R14: 5.1k, Resistor_SMD:R_0402_1005Metric_Pad0.72x0.64mm_HandSolder, F.Cu at (241.2, 100.0)
- added R15: 5.1k, Resistor_SMD:R_0402_1005Metric_Pad0.72x0.64mm_HandSolder, F.Cu at (241.2, 102.0)
- added R16: 5.1k, Resistor_SMD:R_0402_1005Metric_Pad0.72x0.64mm_HandSolder, F.Cu at (241.2, 104.0)
- added R17: 27k, Resistor_SMD:R_0402_1005Metric_Pad0.72x0.64mm_HandSolder, F.Cu at (238.2, 80.1)
- added R18: 10k, Resistor_SMD:R_0402_1005Metric_Pad0.72x0.64mm_HandSolder, F.Cu at (238.2, 82.1)
- added R19: 1k, Resistor_SMD:R_0402_1005Metric_Pad0.72x0.64mm_HandSolder, F.Cu at (238.2, 84.0)
- added R20: 22, Resistor_SMD:R_0402_1005Metric_Pad0.72x0.64mm_HandSolder, F.Cu at (224.9, 90.1)
- added R21: 22, Resistor_SMD:R_0402_1005Metric_Pad0.72x0.64mm_HandSolder, F.Cu at (224.9, 92.1)
- added R22: 22, Resistor_SMD:R_0402_1005Metric_Pad0.72x0.64mm_HandSolder, F.Cu at (224.9, 94.1)
- added R23: 0, Resistor_SMD:R_0402_1005Metric_Pad0.72x0.64mm_HandSolder, F.Cu at (224.9, 96.1)
- added R24: 0, Resistor_SMD:R_0402_1005Metric_Pad0.72x0.64mm_HandSolder, F.Cu at (232.7, 96.0)
- added SW1: Boot, TS24CA Tactile switch:TS24CA, F.Cu at (209.8, 122.8)
- added SW2: PWR, TS24CA Tactile switch:TS24CA, F.Cu at (209.8, 130.3)
- added SW3: NAV, TS24CA Tactile switch:TS24CA, F.Cu at (209.8, 137.8)
- added SW4: UP, TS24CA Tactile switch:TS24CA, F.Cu at (209.8, 145.3)
- added TP1: RXD, TestPoint:TestPoint_Pad_D1.0mm, F.Cu at (221.7, 130.7)
- added TP2: TXD, TestPoint:TestPoint_Pad_D1.0mm, F.Cu at (221.7, 133.7)
- added TP3: 3.3, TestPoint:TestPoint_Pad_D2.0mm, F.Cu at (216.2, 121.1)
- added TP4: SDA, TestPoint:TestPoint_Pad_D2.0mm, F.Cu at (216.2, 125.2)
- added TP5: SCL, TestPoint:TestPoint_Pad_D2.0mm, F.Cu at (216.2, 129.2)
- added TP6: GND, TestPoint:TestPoint_Pad_D2.0mm, F.Cu at (216.2, 133.3)
- added U7: AZ1117-1.8, Package_TO_SOT_SMD:SOT-89-3, F.Cu at (223.6, 122.1)
- C10, C11, C23: footprint Capacitor_SMD:C_1206_3216Metric_Pad1.33x1.80mm_HandSolder -> Capacitor_SMD:C_0402_1005Metric_Pad0.74x0.62mm_HandSolder
- U2: footprint Package_TO_SOT_SMD:SOT-89-3_Handsoldering -> Package_TO_SOT_SMD:SOT-89-3
Connections:
- IC1 pad 6: /ATGM336H/V_GPS -> +3V3
- U10 pad 7: GND -> PWR_KEY_GSM

Commit message: bottom board conn. done
Parts:
- removed ANT1: 1462350001, Molex GPS antenna:ANT_1462350001
- removed C34, C35: NC, Capacitor_SMD:C_0402_1005Metric_Pad0.74x0.62mm_HandSolder
- removed IC1: ATGM336H-5N31, ATGM336H-5N31:ATGM336H5N31
- removed L1: 47nH, Inductor_SMD:L_0402_1005Metric
- removed R12: 5.1k, Resistor_SMD:R_0402_1005Metric_Pad0.72x0.64mm_HandSolder
- removed R24: 0, Resistor_SMD:R_0402_1005Metric_Pad0.72x0.64mm_HandSolder
- removed SW4: UP, TS24CA Tactile switch:TS24CA
- removed U9: M24C32, Package_SO:TSSOP-8_4.4x3mm_P0.65mm
- added C36: 10uF, Capacitor_SMD:C_0402_1005Metric_Pad0.74x0.62mm_HandSolder, F.Cu at (128.6, 87.5)
- added R25: 162k 1%, Resistor_SMD:R_0402_1005Metric_Pad0.72x0.64mm_HandSolder, F.Cu at (128.6, 86.0)
- added R26: 30.1k 1%, Resistor_SMD:R_0402_1005Metric_Pad0.72x0.64mm_HandSolder, F.Cu at (131.2, 86.0)
- added TP7: Bat+, TestPoint:TestPoint_Pad_D1.0mm, F.Cu at (125.0, 73.2)
- added TP8: Bat-, TestPoint:TestPoint_Pad_D1.0mm, F.Cu at (121.6, 70.9)
- C10: value 10uF -> 0.1uF
- C11: value 10uF -> 10pF
- C15: value 10uF -> 100pF
- C20, C21, C29, C30, C31, C32, C33, J5, R14, R15, R16, R20, R21, R22, R23, TP1, TP2, U10, U4: moved to B.Cu
- D1: footprint LED_SMD:LED_0805_2012Metric_Pad1.15x1.40mm_HandSolder -> LED_SMD:LED_0402_1005Metric_Pad0.77x0.64mm_HandSolder
- J2: moved to F.Cu
- JP1: footprint Jumper:SolderJumper-2_P1.3mm_Open_RoundedPad1.0x1.5mm -> Capacitor_SMD:C_0402_1005Metric
- R11: value 5.1k -> DNP/TP
- TP3, TP4, TP5, TP6: footprint TestPoint:TestPoint_Pad_D2.0mm -> TestPoint:TestPoint_Pad_D1.0mm
- U2: value AP1117-33 -> TPS7A7001DDA; footprint Package_TO_SOT_SMD:SOT-89-3 -> Package_SO:TI_SO-PowerPAD-8
- U3: footprint Package_SO:SOIC-8_5.23x5.23mm_P1.27mm -> Package_SON:WSON-8-1EP_6x5mm_P1.27mm_EP3.4x4.3mm
- U8: value 3.3V EN_LDO -> L96; footprint Package_TO_SOT_SMD:SOT-23-5 -> L96 (1):XCVR_L96
- moved R11 140.5 mm to (96.9, 80.3), turned to -90 degrees
- moved R16 131.4 mm to (110.3, 92.3), turned to 90 degrees
- moved R15 130.1 mm to (111.6, 90.3), turned to -90 degrees
- moved C22 127.1 mm to (114.4, 74.5), turned to 180 degrees
- moved C20 126.3 mm to (118.5, 89.7)
- moved TP6 125.0 mm to (97.0, 95.4)
- moved TP5 124.4 mm to (97.0, 93.2)
- moved TP4 123.9 mm to (97.0, 91.0)
- moved R10 123.8 mm to (114.4, 79.5), turned to 180 degrees
- moved Q1 123.1 mm to (119.0, 77.0)
- moved R14 123.0 mm to (118.5, 91.7)
- moved TP3 121.4 mm to (97.0, 97.7)
- moved R19 116.5 mm to (122.0, 76.3), turned to 180 degrees
- moved R18 116.3 mm to (122.0, 77.6), turned to 180 degrees
- moved C17 116.3 mm to (116.9, 92.0), turned to 180 degrees
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Connections:
- C1 pad 1: +3V3 -> VDD_3.3
- C10 pad 1: +BATT -> VDD_3.3_t
- C11 pad 1: +3V3 -> VDD_3.3_t
- C12 pad 1: +3V3 -> VDD_3.3
- C15 pad 1: VDD_3.3 -> VDD_3.3_t
- C16 pad 1: +3V3 -> VDD_3.3
- C18 pad 1: +3V3 -> VDD_3.3
- C2 pad 1: +3V3 -> VDD_3.3
- C23 pad 1: VDD_3.3 -> +BATT
- C29 pad 1: VDD_3.3 -> VDD_3.3_t
- C3 pad 1: +3V3 -> VDD_3.3
- C30 pad 1: VDD_3.3 -> VDD_3.3_t
- C31 pad 1: VDD_3.3 -> VDD_3.3_t
- C4 pad 1: +3V3 -> VDD_3.3
- C5 pad 1: +3V3 -> VDD_3.3
- C6 pad 1: +3V3 -> VDD_3.3
- J3 pad 1: +3V3 -> GSM_RX
- J3 pad 2: PWR_KEY_GSM -> GSM_TX
- J3 pad 3: GPS_RST -> Force_ON
- J3 pad 4: GPS_TXD -> PWR_KEY_GSM
- J3 pad 6: GPS_PPS -> GPS_TXD
- J3 pad 7: GSM_TX -> unconnected-(J3-Pin_7-Pad7)
- J3 pad 8: GSM_RX -> unconnected-(J3-Pin_8-Pad8)
- J4 pad 1: +3V3 -> GSM_RX_t
- J4 pad 2: PWR_KEY_GSM -> GSM_TX_t
- J4 pad 3: GPS_RST -> Force_ON_t
- J4 pad 4: GPS_TXD -> PWR_KEY_GSM_t
- J4 pad 5: GPS_RXD -> GPS_RXD_t
- J4 pad 6: GPS_PPS -> GPS_TXD_t
- J4 pad 7: GSM_TX -> unconnected-(J4-Pin_7-Pad7)
- J4 pad 8: GSM_RX -> unconnected-(J4-Pin_8-Pad8)
- J4 pad 9: VDD_3.3 -> VDD_3.3_t
- JP1 pad 1: +3V3 -> VDD_3.3
- R11 pad 1: MAX30102_SDA -> GND
- R11 pad 2: +3V3 -> Net-(R11-Pad2)
- R14 pad 2: +3V3 -> VDD_3.3
- R15 pad 1: +3V3 -> VDD_3.3
- R16 pad 1: +3V3 -> VDD_3.3
- R3 pad 1: +3V3 -> VDD_3.3
- R4 pad 1: Net-(R4-Pad1) -> Net-(R11-Pad2)
- R5 pad 1: +3V3 -> VDD_3.3
- R9 pad 2: VBUS -> Onboard_LED
- SW1 pad 2: Net-(R4-Pad1) -> NAV_BUTTON_2
- TP3 pad 1: +3V3 -> VDD_3.3
- U1 pad 1: +3V3 -> VDD_3.3
- U1 pad 10: +3V3 -> VDD_3.3
- U1 pad 11: MAX30102_SDA -> unconnected-(U1-GPIO8-Pad11)
- U1 pad 12: MAX30102_SCL -> unconnected-(U1-GPIO9-Pad12)
- U1 pad 13: unconnected-(U1-GPIO10-Pad13) -> Heart_rate_INT
- U1 pad 14: Heart_rate_INT -> Onboard_LED
- U1 pad 16: MPU_INT -> unconnected-(U1-GPIO13-Pad16)
- U1 pad 17: unconnected-(U1-GPIO14-Pad17) -> NAV_BUTTON
- U1 pad 2: unconnected-(U1-GPIO0-Pad2) -> NAV_BUTTON_2
- U1 pad 22: +3V3 -> VDD_3.3
- U1 pad 29: PWR_BUTTON -> Force_ON
- U1 pad 3: unconnected-(U1-GPIO1-Pad3) -> PWR_BUTTON
- U1 pad 30: unconnected-(U1-GPIO19-Pad30) -> PWR_KEY_GSM
- U1 pad 31: NAV_BUTTON -> GPS_RXD
- U1 pad 32: unconnected-(U1-GPIO21-Pad32) -> GPS_TXD
- U1 pad 33: +3V3 -> VDD_3.3
- U1 pad 34: UP_BUTTON -> unconnected-(U1-GPIO22-Pad34)
- U1 pad 35: GPS_PPS -> MPU_INT
- U1 pad 36: GPS_RXD -> MAX30102_SDA
- U1 pad 37: GPS_TXD -> MAX30102_SCL
- U1 pad 38: V_SENSE -> CHARGER_EN
- U1 pad 40: CHARGER_EN -> unconnected-(U1-GPIO28_ADC2-Pad40)
- U1 pad 41: unconnected-(U1-GPIO29_ADC3-Pad41) -> V_SENSE
- U1 pad 42: +3V3 -> VDD_3.3
- U1 pad 43: +3V3 -> VDD_3.3
- U1 pad 44: +3V3 -> VDD_3.3
- U1 pad 48: +3V3 -> VDD_3.3
- U1 pad 49: +3V3 -> VDD_3.3
- U1 pad 8: LDO_EN -> unconnected-(U1-GPIO6-Pad8)
- U1 pad 9: GPS_RST -> unconnected-(U1-GPIO7-Pad9)
- U10 pad 17: GSM_TX -> GSM_TX_t
- U10 pad 18: GSM_RX -> GSM_RX_t
- U10 pad 42: VDD_3.3 -> VDD_3.3_t
- U10 pad 43: VDD_3.3 -> VDD_3.3_t
- U10 pad 7: PWR_KEY_GSM -> PWR_KEY_GSM_t
- U2 pad 1: GND -> unconnected-(U2-NC-Pad1)
- U2 pad 2: +3V3 -> +BATT
- U3 pad 8: +3V3 -> VDD_3.3
- U4 pad 10: +3V3 -> VDD_3.3
- U4 pad 9: +3V3 -> VDD_3.3
- U6 pad 13: +3V3 -> VDD_3.3
- U6 pad 8: +3V3 -> VDD_3.3
- U7 pad 3: +3V3 -> VDD_3.3
- U8 pad 1: +BATT -> (no net)
- U8 pad 2: GND -> unconnected-(U8-3D_FIX-Pad2)
- U8 pad 3: LDO_EN -> unconnected-(U8-I2C_SDA-Pad3)
- U8 pad 4: (no net) -> GND
- U8 pad 5: VDD_3.3 -> GND
Routing:
- net VDD_3.3: track 0.00 -> 50.1 mm, vias 0 -> 32
- net PWR_BUTTON: track 0.00 -> 40.2 mm, vias 0 -> 2
- net NAV_BUTTON_2: track 0.00 -> 31.1 mm, vias 0 -> 2
- net GSM_TX_t: track 0.00 -> 28.0 mm, vias 0 -> 2
- net GSM_RX_t: track 0.00 -> 26.8 mm, vias 0 -> 2
- net GPS_TXD_t: track 0.00 -> 26.7 mm, vias 0 -> 2
- net Heart_rate_INT: track 0.00 -> 26.0 mm, vias 0 -> 1
- net Net-(J2-IO): track 0.00 -> 25.6 mm, vias 0 -> 2
- net Net-(J2-CLK): track 0.00 -> 25.5 mm, vias 0 -> 2
- net GPS_RXD_t: track 0.00 -> 24.6 mm, vias 0 -> 2
- net +BATT: track 0.00 -> 24.3 mm
- net CHARGER_EN: track 0.00 -> 22.1 mm, vias 0 -> 2
- net +1V1: track 0.00 -> 21.9 mm, vias 0 -> 2
- net PWR_KEY_GSM_t: track 0.00 -> 21.5 mm, vias 0 -> 1
- net Net-(J2-RST): track 0.00 -> 21.3 mm, vias 0 -> 2
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- added copper zone on B.Cu, net GND
- added copper zone on F.Cu, net GND
- added copper zone on F.Cu, net VDD_3.3
- added copper zone on In2.Cu, net VDD_3.3
- added copper zone on In2.Cu, net VDD_3.3_t
Other:
- board outline added: 127 x 67.9 mm
- copper layers 2 -> 4

Commit message: Final Design
Parts:
- added E1: NN02-201, NN02-201:XCVR_NN02-201, B.Cu at (198.0, 92.9)
- added R12: 0, Resistor_SMD:R_0402_1005Metric_Pad0.72x0.64mm_HandSolder, B.Cu at (198.0, 85.4)
- added R24: 0, Resistor_SMD:R_0402_1005Metric_Pad0.72x0.64mm_HandSolder, B.Cu at (198.0, 86.6)
- added kibuzzard-648D8F43: G***, kibuzzard-648D8F43, F.Cu at (106.1, 97.9)
- added kibuzzard-648D8F93: G***, kibuzzard-648D8F93, F.Cu at (139.6, 90.4)
- added kibuzzard-648D8FB3: G***, kibuzzard-648D8FB3, F.Cu at (117.3, 110.1)
- added kibuzzard-648D8FC5: G***, kibuzzard-648D8FC5, F.Cu at (117.6, 71.1)
- added kibuzzard-648D902E: G***, kibuzzard-648D902E, F.Cu at (128.8, 97.0)
- added kibuzzard-648D909E: G***, kibuzzard-648D909E, F.Cu at (106.5, 80.7)
- added kibuzzard-648D90C6: G***, kibuzzard-648D90C6, F.Cu at (139.8, 81.5)
- added kibuzzard-648D90E2: G***, kibuzzard-648D90E2, F.Cu at (124.0, 81.7)
- added kibuzzard-648D9126: G***, kibuzzard-648D9126, B.Cu at (123.0, 86.4)
- added kibuzzard-648D91AF: G***, kibuzzard-648D91AF, F.Cu at (135.4, 103.9)
- added kibuzzard-648D920B: G***, kibuzzard-648D920B, F.Cu at (130.3, 74.9)
- added kibuzzard-648D921A: G***, kibuzzard-648D921A, F.Cu at (126.4, 71.9)
- added kibuzzard-648D92FA: G***, kibuzzard-648D92FA, F.Cu at (167.0, 80.3)
- added kibuzzard-648D9334: G***, kibuzzard-648D9334, B.Cu at (165.0, 94.3)
- added kibuzzard-648D9374: G***, kibuzzard-648D9374, B.Cu at (165.0, 84.4)
- added kibuzzard-648D9446: G***, kibuzzard-648D9446, F.Cu at (101.9, 91.3)
- added kibuzzard-648D944C: G***, kibuzzard-648D944C, F.Cu at (102.0, 93.5)
- Q1: value HSSN3134 -> BSS214
- SW1: value Boot -> NAV2; footprint TS24CA Tactile switch:TS24CA -> TL3330AF260QG:SW_TL3330AF260QG
- SW2, SW3: footprint TS24CA Tactile switch:TS24CA -> TL3330AF260QG:SW_TL3330AF260QG
- U7: value AZ1117-1.8 -> AP2127K-1.8; footprint Package_TO_SOT_SMD:SOT-89-3 -> Package_TO_SOT_SMD:SOT-23-5
- moved J5 15.7 mm to (198.0, 80.2), turned to 180 degrees
- moved TP1 12.8 mm to (165.0, 87.8)
- moved C33 7.96 mm to (193.0, 85.5), turned to 90 degrees
- moved SW1 7.09 mm to (122.2, 70.3), turned to 180 degrees
- moved R11 7.06 mm to (103.9, 81.2)
- moved SW3 7.02 mm to (122.2, 110.5), turned to 0 degrees
- moved C1 7.01 mm to (108.0, 95.5)
- moved C12 7.01 mm to (110.3, 82.4)
- moved C13 7.01 mm to (110.3, 102.8)
- moved C14 7.01 mm to (112.7, 102.8)
- moved C17 7.01 mm to (123.9, 92.3)
- moved C18 7.01 mm to (133.4, 94.2)
- moved C19 7.01 mm to (133.4, 92.3)
- moved C2 7.01 mm to (120.9, 91.9)
- moved C20 7.01 mm to (125.5, 90.0)
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Connections:
- C32 pad 1: Net-(J5-SIG) -> Net-(C32-Pad1)
- R23 pad 2: Net-(J5-SIG) -> Net-(C32-Pad1)
- U7 pad 1: GND -> VDD_3.3
- U7 pad 2: +1V8 -> GND
Routing:
- net Net-(U10-DBG_RXD): track 0.00 -> 22.4 mm
- net Net-(U10-DBG_TXD): track 0.00 -> 22.2 mm
- net NAV_BUTTON_2: track 31.1 -> 26.2 mm
- net VDD_3.3: track 50.1 -> 54.4 mm, vias 32 -> 34
- net Net-(U10-RF_ANT): track 0.00 -> 3.65 mm
- net Net-(E1-Pad1): track 0.00 -> 3.30 mm
- net Net-(J5-SIG): track 0.00 -> 3.08 mm
- net Net-(C32-Pad1): track 0.00 -> 2.70 mm
- net VDD_3.3_t: track 9.92 -> 7.65 mm, vias 3 -> 12
- net NAV_BUTTON: track 17.6 -> 19.1 mm
- net PWR_BUTTON: track 40.2 -> 41.3 mm
- net Net-(U8-RF_IN): track 0.00 -> 1.00 mm
- net Net-(R11-Pad2): track 2.09 -> 1.49 mm
- net GND: vias 92 -> 106
- added copper zone on B.Cu, net Net-(E1-Pad1)
- added copper zone on B.Cu, net Net-(J5-SIG)
- added copper zone on B.Cu, net VDD_3.3_t
- added copper zone on F.Cu, net VDD_3.3_t
Other:
- board size 127 x 67.9 mm -> 124.7 x 64.3 mm
