File: charging_circuit&pwr_reg.kicad_sch (KiCad schematic)
At the start: 13 parts, among them Q1 HSSN3134, U3 AP1117-33, U5 MCP73831-2-OT, U8 3.3V EN_LDO

Commit message: assigned footprints and checked the schematic
Parts:
- C13, C15: footprint Capacitor_SMD:C_1206_3216Metric_Pad1.33x1.80mm_HandSolder -> Capacitor_SMD:C_0402_1005Metric_Pad0.74x0.62mm_HandSolder
- C22: footprint (none) -> Capacitor_SMD:C_0402_1005Metric_Pad0.74x0.62mm_HandSolder
- Q1: footprint (none) -> Package_TO_SOT_SMD:SOT-323_SC-70
- R10, R13, R17, R18, R19: footprint (none) -> Resistor_SMD:R_0402_1005Metric_Pad0.72x0.64mm_HandSolder
- U3: footprint Package_TO_SOT_SMD:SOT-89-3_Handsoldering -> Package_TO_SOT_SMD:SOT-89-3
Connections:
- net GND: now also Q1.2 (S); no longer Q1.3 (S)
- net at Q1.1 (G): now also R18.2, R19.2; no longer U5.2 (V_{SS})
- new net: Q1.3 (D), U5.2 (V_{SS})
Changed lines of the file:
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@@
       (effects (font (size 1.27 1.27)) (justify left))
     )
-    (property "Footprint" "" (at 161.29 58.928 90)
+    (property "Footprint" "Resistor_SMD:R_0402_1005Metric_Pad0.72x0.64mm_HandSolder" (at 161.29 58.928 90)
       (effects (font (size 1.27 1.27)) hide)
     )
@@
       (effects (font (size 1.27 1.27)))
     )
-    (property "Footprint" "Package_TO_SOT_SMD:SOT-89-3_Handsoldering" (at 119.126 114.808 0)
+    (property "Footprint" "Package_TO_SOT_SMD:SOT-89-3" (at 119.126 114.808 0)
       (effects (font (size 1.27 1.27)) hide)
     )
@@
       (effects (font (size 1.27 1.27)) (justify left))
     )
-    (property "Footprint" "" (at 182.88 67.31 0)
+    (property "Footprint" "Package_TO_SOT_SMD:SOT-323_SC-70" (at 182.88 67.31 0)
       (effects (font (size 1.27 1.27)) hide)
     )
@@
       (effects (font (size 1.27 1.27)) (justify left))
     )
-    (property "Footprint" "" (at 171.958 76.2 90)
+    (property "Footprint" "Resistor_SMD:R_0402_1005Metric_Pad0.72x0.64mm_HandSolder" (at 171.958 76.2 90)
       (effects (font (size 1.27 1.27)) hide)
     )
@@
       (effects (font (size 1.27 1.27)))
     )
-    (property "Footprint" "" (at 98.552 67.31 90)
+    (property "Footprint" "Resistor_SMD:R_0402_1005Metric_Pad0.72x0.64mm_HandSolder" (at 98.552 67.31 90)
       (effects (font (size 1.27 1.27)) hide)
     )
@@
       (effects (font (size 1.27 1.27)) (justify left))
     )
-    (property "Footprint" "" (at 162.56 71.628 90)
+    (property "Footprint" "Resistor_SMD:R_0402_1005Metric_Pad0.72x0.64mm_HandSolder" (at 162.56 71.628 90)
       (effects (font (size 1.27 1.27)) hide)
     )
@@
       (effects (font (size 1.27 1.27)))
     )
-    (property "Footprint" "" (at 98.552 54.61 90)
+    (property "Footprint" "Resistor_SMD:R_0402_1005Metric_Pad0.72x0.64mm_HandSolder" (at 98.552 54.61 90)
       (effects (font (size 1.27 1.27)) hide)
     )
@@
       (effects (font (size 1.27 1.27)) (justify left))
     )
-    (property "Footprint" "Capacitor_SMD:C_1206_3216Metric_Pad1.33x1.80mm_HandSolder" (at 177.4952 130.81 0)
+    (property "Footprint" "Capacitor_SMD:C_0402_1005Metric_Pad0.74x0.62mm_HandSolder" (at 177.4952 130.81 0)
       (effects (font (size 1.27 1.27)) hide)
     )
@@
       (effects (font (size 1.27 1.27)) (justify left))
     )
-    (property "Footprint" "Capacitor_SMD:C_1206_3216Metric_Pad1.33x1.80mm_HandSolder" (at 106.1212 128.778 0)
+    (property "Footprint" "Capacitor_SMD:C_0402_1005Metric_Pad0.74x0.62mm_HandSolder" (at 106.1212 128.778 0)
       (effects (font (size 1.27 1.27)) hide)
     )
@@
       (effects (font (size 1.27 1.27)) (justify left))
     )
-    (property "Footprint" "Capacitor_SMD:C_1206_3216Metric_Pad1.33x1.80mm_HandSolder" (at 132.7912 128.778 0)
+    (property "Footprint" "Capacitor_SMD:C_0402_1005Metric_Pad0.74x0.62mm_HandSolder" (at 132.7912 128.778 0)
       (effects (font (size 1.27 1.27)) hide)
     )
@@
       (effects (font (size 1.27 1.27)) (justify right))
     )
-    (property "Footprint" "" (at 160.3248 40.64 0)
-      (effects (font (size 1.27 1.27)) hide)
-    )
+    (property "Footprint" "Capacitor_SMD:C_0402_1005Metric_Pad0.74x0.62mm_HandSolder" (at 160.3248 40.64 0)
+      (effects (font (size 1.27 1.27)) hide)
+    )

Commit message: bottom board conn. done
Parts:
- removed C13, C15 (x2): 10uF, Capacitor_SMD:C_0402_1005Metric_Pad0.74x0.62mm_HandSolder, symbol Device:C
- removed U3: AP1117-33, Package_TO_SOT_SMD:SOT-89-3, symbol Regulator_Linear:AP1117-33
- removed U8: 3.3V EN_LDO, Package_TO_SOT_SMD:SOT-23-5, symbol PJ9193M33SE:PJ9193_3.3V
- added C23, C36: 10uF, Capacitor_SMD:C_0402_1005Metric_Pad0.74x0.62mm_HandSolder, symbol Device:C
- added R25: 162k 1%, Resistor_SMD:R_0402_1005Metric_Pad0.72x0.64mm_HandSolder, symbol Device:R
- added R26: 30.1k 1%, Resistor_SMD:R_0402_1005Metric_Pad0.72x0.64mm_HandSolder, symbol Device:R
- added TP7: Bat+, TestPoint:TestPoint_Pad_D1.0mm, symbol Connector:TestPoint
- added TP8: Bat-, TestPoint:TestPoint_Pad_D1.0mm, symbol Connector:TestPoint
- added U2: TPS7A7001DDA, Package_SO:TI_SO-PowerPAD-8, symbol Regulator_Linear:TPS7A7001DDA
Connections:
- net +3V3: now also C36.1, R25.1, U2.6 (OUT)
- net +BATT: now also C23.1, TP7.1, U2.2 (EN), U2.3 (IN)
- net GND: now also C23.2, C36.2, R26.2, TP8.1, U2.8 (GND), U2.9 (EP)
- new net: R25.2, R26.1, U2.7 (FB)
Other:
- moved on the sheet: R13, R17

Commit message: Final Design
Parts:
- Q1: value HSSN3134 -> BSS214
Changed lines of the file:
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@@
       (effects (font (size 1.27 1.27)) (justify left))
     )
-    (property "Value" "HSSN3134" (at 184.15 71.755 0)
+    (property "Value" "BSS214" (at 184.15 71.755 0)
       (effects (font (size 1.27 1.27)) (justify left))
     )
