File: quectelm66.kicad_sch (KiCad schematic)
At the start: 19 parts, among them J2 SIM8060-6-0-14-00-A, U10 M66

Commit message: assigned footprints and checked the schematic
Parts:
- removed AE1: 900MHz, symbol Device:Antenna_Chip
- added J5: U.FL-R-SMT-1(10), U.FL-R-SMT-1_10_:HRS_U.FL-R-SMT-1(10), symbol U.FL-R-SMT-1_10_:U.FL-R-SMT-1(10)
- C24, C25, C26, C27, C28, C30, C31, C32, C33: footprint (none) -> Capacitor_SMD:C_0402_1005Metric_Pad0.74x0.62mm_HandSolder
- C29: footprint (none) -> Capacitor_Tantalum_SMD:CP_EIA-7343-30_AVX-N
- R20, R21, R22, R23: footprint (none) -> Resistor_SMD:R_0402_1005Metric_Pad0.72x0.64mm_HandSolder
- TP1, TP2: footprint (none) -> TestPoint:TestPoint_Pad_D1.0mm
- U10: footprint XCVR_M66 -> Quectel M66:XCVR_M66
Connections:
- net GND: now also J5.1 (GND), J5.3 (GND)
- net at C32.1, R23.2: now also J5.2 (SIG)

Commit message: bottom board conn. done
Connections:
- net GSM_RX renamed GSM_RX_t
- net GSM_TX renamed GSM_TX_t
- net PWR_KEY_GSM renamed PWR_KEY_GSM_t
- net VDD_3.3 renamed VDD_3.3_t
Other:
- note added: "*add ceramic antenna*"
Changed lines of the file:
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@@
     (stroke (width 0) (type default))
+  )
+  (text "*add ceramic antenna*" (at 116.84 125.73 0)
+    (effects (font (size 3 3) (thickness 0.254) bold) (justify left bottom))
   )
   (label "SIM_RST" (at 158.75 99.06 180) (fields_autoplaced)
@@
     (effects (font (size 1 1)) (justify left bottom))
   )
-  (global_label "VDD_3.3" (shape input) (at 101.6 64.77 90) (fields_autoplaced)
+  (global_label "PWR_KEY_GSM_t" (shape input) (at 50.8 86.36 180) (fields_autoplaced)
+    (effects (font (size 1 1)) (justify right))
+    (property "Intersheetrefs" "${INTERSHEET_REFS}" (at 36.6549 86.36 0)
+      (effects (font (size 1.27 1.27)) (justify right) hide)
+    )
+  )
+  (global_label "GSM_RX_t" (shape output) (at 50.8 101.6 180) (fields_autoplaced)
+    (effects (font (size 1 1) (color 88 18 132 1)) (justify right))
+    (property "Intersheetrefs" "${INTERSHEET_REFS}" (at 41.3692 101.6 0)
+      (effects (font (size 1.27 1.27)) (justify right) hide)
+    )
+  )
+  (global_label "VDD_3.3_t" (shape input) (at 147.32 64.77 180) (fields_autoplaced)
+    (effects (font (size 1 1) (color 255 149 14 1)) (justify right))
+    (property "Intersheetrefs" "${INTERSHEET_REFS}" (at 137.6988 64.77 0)
+      (effects (font (size 1.27 1.27)) (justify right) hide)
+    )
+  )
+  (global_label "VDD_3.3_t" (shape input) (at 101.6 64.77 90) (fields_autoplaced)
     (effects (font (size 1 1) (color 255 149 14 1)) (justify left))
-    (property "Intersheetrefs" "${INTERSHEET_REFS}" (at 101.6 56.4821 90)
+    (property "Intersheetrefs" "${INTERSHEET_REFS}" (at 101.6 55.1488 90)
       (effects (font (size 1.27 1.27)) (justify left) hide)
     )
   )
-  (global_label "PWR_KEY_GSM" (shape input) (at 50.8 86.36 180) (fields_autoplaced)
-    (effects (font (size 1 1)) (justify right))
-    (property "Intersheetrefs" "${INTERSHEET_REFS}" (at 37.9882 86.36 0)
+  (global_label "GSM_TX_t" (shape output) (at 50.8 99.06 180) (fields_autoplaced)
+    (effects (font (size 1 1) (color 88 18 132 1)) (justify right))
+    (property "Intersheetrefs" "${INTERSHEET_REFS}" (at 41.6073 99.06 0)
       (effects (font (size 1.27 1.27)) (justify right) hide)
     )
-  )
-  (global_label "GSM_TX" (shape output) (at 50.8 99.06 180) (fields_autoplaced)
-    (effects (font (size 1 1) (color 88 18 132 1)) (justify right))
-    (property "Intersheetrefs" "${INTERSHEET_REFS}" (at 42.9406 99.06 0)
-      (effects (font (size 1.27 1.27)) (justify right) hide)
-    )
-  )
-  (global_label "VDD_3.3" (shape input) (at 147.32 64.77 0) (fields_autoplaced)
-    (effects (font (size 1 1) (color 255 149 14 1)) (justify left))
-    (property "Intersheetrefs" "${INTERSHEET_REFS}" (at 155.6079 64.77 0)
-      (effects (font (size 1.27 1.27)) (justify left) hide)
-    )
-  )
-  (global_label "GSM_RX" (shape output) (at 50.8 101.6 180) (fields_autoplaced)
-    (effects (font (size 1 1) (color 88 18 132 1)) (justify right))
-    (property "Intersheetrefs" "${INTERSHEET_REFS}" (at 42.7025 101.6 0)
-      (effects (font (size 1.27 1.27)) (justify right) hide)
-    )

Commit message: Final Design
Parts:
- added E1: NN02-201, NN02-201:XCVR_NN02-201, symbol NN02-201:NN02-201
- added R12, R24: 0, Resistor_SMD:R_0402_1005Metric_Pad0.72x0.64mm_HandSolder, symbol Device:R
Connections:
- net at C32.1, R23.2: now also R12.1, R24.1; no longer J5.2 (SIG)
- new net: J5.2 (SIG), R12.2
- new net: E1.1, R24.2
Other:
- note removed: "*add ceramic antenna*"
- moved on the sheet: C24, C25, C26, C27, C28, C29, C30, C31, C32, C33, J2, J5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
